File: DG-Board.kicad_pcb (KiCad board)
At the start: 2 copper layers, 1 part, among them U1 DG_Bus

Commit message: Fixed DG-Bus footprint. Changed Margin to Edge.Cuts. Changed F.CrtYd to F.SilkS.
Other:
- board outline added: 381 x 382.3 mm
